File: template_project_kicad.kicad_pcb (KiCad board)
At the start: 2 copper layers, 53.3 x 50.8 mm, 5 parts

Commit message: Assigned GND net to copper zones
Connections:
- A1 pad 13: unconnected-(A1-GND-Pad13) -> /GND
- A1 pad 18: unconnected-(A1-GND-Pad18) -> /GND
- A1 pad 23: unconnected-(A1-GND-Pad23) -> /GND
- A1 pad 28: unconnected-(A1-GND-Pad28) -> /GND
- A1 pad 3: unconnected-(A1-GND-Pad3) -> /GND
- A1 pad 33: unconnected-(A1-GND|AGND-Pad33) -> /GND
- A1 pad 38: unconnected-(A1-GND-Pad38) -> /GND
- A1 pad 8: unconnected-(A1-GND-Pad8) -> /GND
Routing:
- added copper zone on B.Cu, net /GND
- added copper zone on F.Cu, net /GND
- removed copper zone on B.Cu, net (none)
- removed copper zone on F.Cu, net (none)
